File: MicroMouse.sch (EAGLE design)
At the start: 63 parts

Commit message: Add files via upload
Other:
- note added: "Buttons"
- note added: "Microcontroller"
- note removed: "BUttons"
Changed lines of the file:
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@@
 <text x="-96.52" y="93.98" size="1.27" layer="91">Communication</text>
 <text x="-111.76" y="-55.88" size="1.27" layer="91">Motor Control</text>
-<text x="-121.92" y="10.16" size="1.27" layer="91">BUttons</text>
+<text x="-124.46" y="10.16" size="1.27" layer="91">Buttons</text>
 <text x="-241.3" y="99.06" size="1.27" layer="91">Emitters</text>
 <text x="-241.3" y="35.56" size="1.27" layer="91">Receiver</text>
 <text x="-241.3" y="-27.94" size="1.27" layer="91">Voltmeter</text>
+<text x="-284.48" y="-66.04" size="1.27" layer="91">Microcontroller</text>
 </plain>
 <instances>
@@
 <net name="N$2" class="0">
 <segment>
-<wire x1="-33.02" y1="101.6" x2="101.6" y2="101.6" width="0.1524" layer="91"/>
-<wire x1="101.6" y1="101.6" x2="99.06" y2="15.24" width="0.1524" layer="91"/>
+<wire x1="-33.02" y1="101.6" x2="99.06" y2="101.6" width="0.1524" layer="91"/>
+<wire x1="99.06" y1="101.6" x2="99.06" y2="15.24" width="0.1524" layer="91"/>
 <wire x1="99.06" y1="15.24" x2="-33.02" y2="15.24" width="0.1524" layer="91"/>
 <wire x1="-33.02" y1="15.24" x2="-33.02" y2="101.6" width="0.1524" layer="91"/>
@@
 <wire x1="99.06" y1="15.24" x2="99.06" y2="-50.8" width="0.1524" layer="91"/>
 <wire x1="-129.54" y1="101.6" x2="-33.02" y2="101.6" width="0.1524" layer="91"/>
-<wire x1="-129.54" y1="101.6" x2="-129.54" y2="15.24" width="0.1524" layer="91"/>
+<wire x1="-129.54" y1="101.6" x2="-129.54" y2="40.64" width="0.1524" layer="91"/>
+<wire x1="-129.54" y1="40.64" x2="-129.54" y2="15.24" width="0.1524" layer="91"/>
 <wire x1="-129.54" y1="15.24" x2="-33.02" y2="15.24" width="0.1524" layer="91"/>
 <wire x1="-33.02" y1="-50.8" x2="-129.54" y2="-50.8" width="0.1524" layer="91"/>
-<wire x1="-129.54" y1="-50.8" x2="-129.54" y2="-177.8" width="0.1524" layer="91"/>
+<wire x1="-129.54" y1="-53.34" x2="-129.54" y2="-177.8" width="0.1524" layer="91"/>
 <wire x1="-129.54" y1="-177.8" x2="99.06" y2="-177.8" width="0.1524" layer="91"/>
 <wire x1="99.06" y1="-177.8" x2="99.06" y2="-50.8" width="0.1524" layer="91"/>
-<wire x1="-129.54" y1="-50.8" x2="-129.54" y2="15.24" width="0.1524" layer="91"/>
-<wire x1="-129.54" y1="101.6" x2="-284.48" y2="101.6" width="0.1524" layer="91"/>
-<wire x1="-284.48" y1="101.6" x2="-294.64" y2="-177.8" width="0.1524" layer="91"/>
-<wire x1="-294.64" y1="-177.8" x2="-129.54" y2="-177.8" width="0.1524" layer="91"/>
+<wire x1="-129.54" y1="-50.8" x2="-129.54" y2="-22.86" width="0.1524" layer="91"/>
+<wire x1="-129.54" y1="-22.86" x2="-129.54" y2="15.24" width="0.1524" layer="91"/>
+<wire x1="-129.54" y1="101.6" x2="-297.18" y2="101.6" width="0.1524" layer="91"/>
+<wire x1="-297.18" y1="101.6" x2="-297.18" y2="40.64" width="0.1524" layer="91"/>
+<wire x1="-297.18" y1="40.64" x2="-297.18" y2="-22.86" width="0.1524" layer="91"/>
+<wire x1="-297.18" y1="-22.86" x2="-297.18" y2="-50.8" width="0.1524" layer="91"/>
+<wire x1="-297.18" y1="-50.8" x2="-297.18" y2="-177.8" width="0.1524" layer="91"/>
+<wire x1="-297.18" y1="-177.8" x2="-129.54" y2="-177.8" width="0.1524" layer="91"/>
+<wire x1="-297.18" y1="40.64" x2="-129.54" y2="40.64" width="0.1524" layer="91"/>
+<junction x="-297.18" y="40.64"/>
+<junction x="-129.54" y="40.64"/>
+<wire x1="-297.18" y1="-22.86" x2="-129.54" y2="-22.86" width="0.1524" layer="91"/>
+<junction x="-297.18" y="-22.86"/>
+<junction x="-129.54" y="-22.86"/>
+<wire x1="-297.18" y1="-50.8" x2="-129.54" y2="-50.8" width="0.1524" layer="91"/>
+<wire x1="-129.54" y1="-50.8" x2="-129.54" y2="-53.34" width="0.1524" layer="91"/>
+<junction x="-297.18" y="-50.8"/>
 </segment>
 </net>

Commit message: Final Schematics
Other:
- note added: "Dream Team"
- note added: "UCSD Micromouse 2017-2018 Sean Liu, Gun Park, Yuqian Cheng, Patrick Lee"
Changed lines of the file:
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@@
 <sheet>
 <plain>
-<text x="-27.94" y="93.98" size="1.778" layer="91">Power Supply</text>
-<text x="-27.94" y="7.62" size="1.778" layer="91">LEDs</text>
-<text x="-96.52" y="93.98" size="1.27" layer="91">Communication</text>
-<text x="-111.76" y="-55.88" size="1.27" layer="91">Motor Control</text>
-<text x="-124.46" y="10.16" size="1.27" layer="91">Buttons</text>
-<text x="-241.3" y="99.06" size="1.27" layer="91">Emitters</text>
-<text x="-241.3" y="35.56" size="1.27" layer="91">Receiver</text>
-<text x="-241.3" y="-27.94" size="1.27" layer="91">Voltmeter</text>
-<text x="-284.48" y="-66.04" size="1.27" layer="91">Microcontroller</text>
+<text x="-25.4" y="86.36" size="7.62" layer="95">Power Supply</text>
+<text x="60.96" y="-7.62" size="7.62" layer="95">LEDs</text>
+<text x="-116.84" y="83.82" size="7.62" layer="95">Communication</text>
+<text x="-2.54" y="-104.14" size="7.62" layer="95">Motor Control</text>
+<text x="-289.56" y="86.36" size="7.62" layer="95">Emitters</text>
+<text x="-287.02" y="25.4" size="7.62" layer="95">Receiver</text>
+<text x="-292.1" y="-35.56" size="7.62" layer="95">Voltmeter</text>
+<text x="-200.66" y="-60.96" size="7.62" layer="95">Microcontroller</text>
+<text x="-124.46" y="5.08" size="7.62" layer="95">Buttons</text>
+<text x="-2.54" y="-170.18" size="10.16" layer="95">Dream Team</text>
+<text x="2.54" y="-180.34" size="2.54" layer="95">UCSD Micromouse 2017-2018
+Sean Liu, Gun Park, Yuqian Cheng, Patrick Lee</text>
 </plain>
 <instances>
@@
 <wire x1="-129.54" y1="15.24" x2="-33.02" y2="15.24" width="0.1524" layer="91"/>
 <wire x1="-33.02" y1="-50.8" x2="-129.54" y2="-50.8" width="0.1524" layer="91"/>
-<wire x1="-129.54" y1="-53.34" x2="-129.54" y2="-177.8" width="0.1524" layer="91"/>
-<wire x1="-129.54" y1="-177.8" x2="99.06" y2="-177.8" width="0.1524" layer="91"/>
-<wire x1="99.06" y1="-177.8" x2="99.06" y2="-50.8" width="0.1524" layer="91"/>
+<wire x1="-129.54" y1="-50.8" x2="-129.54" y2="-182.88" width="0.1524" layer="91"/>
+<wire x1="-129.54" y1="-182.88" x2="-5.08" y2="-182.88" width="0.1524" layer="91"/>
+<wire x1="-5.08" y1="-182.88" x2="99.06" y2="-182.88" width="0.1524" layer="91"/>
+<wire x1="99.06" y1="-182.88" x2="99.06" y2="-157.48" width="0.1524" layer="91"/>
+<wire x1="99.06" y1="-157.48" x2="99.06" y2="-50.8" width="0.1524" layer="91"/>
 <wire x1="-129.54" y1="-50.8" x2="-129.54" y2="-22.86" width="0.1524" layer="91"/>
 <wire x1="-129.54" y1="-22.86" x2="-129.54" y2="15.24" width="0.1524" layer="91"/>
@@
 <wire x1="-297.18" y1="40.64" x2="-297.18" y2="-22.86" width="0.1524" layer="91"/>
 <wire x1="-297.18" y1="-22.86" x2="-297.18" y2="-50.8" width="0.1524" layer="91"/>
-<wire x1="-297.18" y1="-50.8" x2="-297.18" y2="-177.8" width="0.1524" layer="91"/>
-<wire x1="-297.18" y1="-177.8" x2="-129.54" y2="-177.8" width="0.1524" layer="91"/>
+<wire x1="-297.18" y1="-50.8" x2="-297.18" y2="-182.88" width="0.1524" layer="91"/>
+<wire x1="-297.18" y1="-182.88" x2="-129.54" y2="-182.88" width="0.1524" layer="91"/>
 <wire x1="-297.18" y1="40.64" x2="-129.54" y2="40.64" width="0.1524" layer="91"/>
 <junction x="-297.18" y="40.64"/>
@@
 <junction x="-129.54" y="-22.86"/>
 <wire x1="-297.18" y1="-50.8" x2="-129.54" y2="-50.8" width="0.1524" layer="91"/>
-<wire x1="-129.54" y1="-50.8" x2="-129.54" y2="-53.34" width="0.1524" layer="91"/>
 <junction x="-297.18" y="-50.8"/>
+<wire x1="-5.08" y1="-182.88" x2="-5.08" y2="-157.48" width="0.1524" layer="91"/>
+<wire x1="-5.08" y1="-157.48" x2="99.06" y2="-157.48" width="0.1524" layer="91"/>
 </segment>
 </net>
@@
 </drawing>
 <compatibility>
+<note version="6.3" minversion="6.2.2" severity="warning">
+Since Version 6.2.2 text objects can contain more than one line,
+which will not be processed correctly with this version.
+</note>
 <note version="8.2" severity="warning">
 Since Version 8.2, EAGLE supports online libraries. The ids

Commit message: Changed 47uF capacitor
Parts:
- C1, C2, C3: device SparkFun-Capacitors:47UF-POLAR-EIA3528-10V-10% -> CAP_TANT_1210IN_3528MM:CAP_TANT_1210IN_3528MM
Changed lines of the file:
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@@
 <part name="BAT_JST-PH" library="BATT_JST-PH_3PIN" deviceset="3PIN" device=""/>
 <part name="REG_3V3_SPX3940" library="REG_3V3_LM3940" deviceset="3V3_REG" device=""/>
-<part name="C1" library="SparkFun-Capacitors" library_urn="urn:adsk.eagle:library:510" deviceset="47UF-POLAR" device="-EIA3528-10V-10%" package3d_urn="urn:adsk.eagle:package:37411/1" value="47uF"/>
-<part name="C2" library="SparkFun-Capacitors" library_urn="urn:adsk.eagle:library:510" deviceset="47UF-POLAR" device="-EIA3528-10V-10%" package3d_urn="urn:adsk.eagle:package:37411/1" value="47uF"/>
-<part name="C3" library="SparkFun-Capacitors" library_urn="urn:adsk.eagle:library:510" deviceset="47UF-POLAR" device="-EIA3528-10V-10%" package3d_urn="urn:adsk.eagle:package:37411/1" value="47uF"/>
 <part name="C11" library="SparkFun-Capacitors" library_urn="urn:adsk.eagle:library:510" deviceset="10UF" device="-0805-10V-10%" package3d_urn="urn:adsk.eagle:package:37429/1" value="10uF"/>
 <part name="GND1" library="SUPPLY" deviceset="GND" device=""/>
@@
 <part name="C9" library="CAP_CERAMIC_0805IN_2012MM" deviceset="CAP_CERAMIC_0805IN_2012MM" device="" value="2.2uF"/>
 <part name="C10" library="CAP_CERAMIC_0805IN_2012MM" deviceset="CAP_CERAMIC_0805IN_2012MM" device="" value="0.1uF"/>
+<part name="C1" library="CAP_TANT_1210IN_3528MM" deviceset="CAP_TANT_1210IN_3528MM" device="" value="47uF"/>
+<part name="C2" library="CAP_TANT_1210IN_3528MM" deviceset="CAP_TANT_1210IN_3528MM" device="" value="47uF"/>
+<part name="C3" library="CAP_TANT_1210IN_3528MM" deviceset="CAP_TANT_1210IN_3528MM" device="" value="47uF"/>
 </parts>
 <sheets>
@@
 <instance part="BAT_JST-PH" gate="G$1" x="-15.24" y="38.1" rot="R90"/>
 <instance part="REG_3V3_SPX3940" gate="G$1" x="66.04" y="60.96"/>
-<instance part="C1" gate="G$1" x="7.62" y="38.1"/>
-<instance part="C2" gate="G$1" x="45.72" y="38.1"/>
-<instance part="C3" gate="G$1" x="83.82" y="38.1"/>
 <instance part="C11" gate="G$1" x="55.88" y="35.56"/>
 <instance part="GND1" gate="1" x="27.94" y="22.86"/>
@@
 <instance part="C9" gate="G$1" x="-193.04" y="-165.1"/>
 <instance part="C10" gate="G$1" x="-167.64" y="-165.1"/>
+<instance part="C1" gate="G$1" x="7.62" y="38.1"/>
+<instance part="C2" gate="G$1" x="45.72" y="38.1"/>
+<instance part="C3" gate="G$1" x="83.82" y="38.1"/>
 </instances>
 <busses>
@@
 <net name="N$3" class="0">
 <segment>
-<pinref part="C1" gate="G$1" pin="+"/>
 <wire x1="7.62" y1="40.64" x2="7.62" y2="60.96" width="0.1524" layer="91"/>
 <wire x1="7.62" y1="60.96" x2="0" y2="60.96" width="0.1524" layer="91"/>
@@
 <wire x1="7.62" y1="60.96" x2="20.32" y2="60.96" width="0.1524" layer="91"/>
 <junction x="7.62" y="60.96"/>
+<pinref part="C1" gate="G$1" pin="+"/>
 </segment>
 </net>
@@
 <wire x1="-12.7" y1="33.02" x2="-12.7" y2="30.48" width="0.1524" layer="91"/>
 <wire x1="-12.7" y1="30.48" x2="7.62" y2="30.48" width="0.1524" layer="91"/>
-<pinref part="C1" gate="G$1" pin="-"/>
 <wire x1="7.62" y1="30.48" x2="7.62" y2="33.02" width="0.1524" layer="91"/>
 <wire x1="7.62" y1="30.48" x2="27.94" y2="30.48" width="0.1524" layer="91"/>
 <junction x="7.62" y="30.48"/>
-<pinref part="C2" gate="G$1" pin="-"/>
 <wire x1="27.94" y1="30.48" x2="45.72" y2="30.48" width="0.1524" layer="91"/>
 <wire x1="45.72" y1="30.48" x2="45.72" y2="33.02" width="0.1524" layer="91"/>
@@
 <wire x1="27.94" y1="53.34" x2="27.94" y2="30.48" width="0.1524" layer="91"/>
 <junction x="27.94" y="30.48"/>
-<pinref part="C3" gate="G$1" pin="-"/>
 <wire x1="55.88" y1="30.48" x2="66.04" y2="30.48" width="0.1524" layer="91"/>
 <wire x1="66.04" y1="30.48" x2="83.82" y2="30.48" width="0.1524" layer="91"/>
@@
 <wire x1="27.94" y1="30.48" x2="27.94" y2="25.4" width="0.1524" layer="91"/>
 <pinref part="GND1" gate="1" pin="GND"/>
+<pinref part="C1" gate="G$1" pin="-"/>
+<pinref part="C2" gate="G$1" pin="-"/>
+<pinref part="C3" gate="G$1" pin="-"/>
 </segment>
 <segment>
@@
 <pinref part="REG_3V3_SPX3940" gate="G$1" pin="IN"/>
 <wire x1="35.56" y1="60.96" x2="45.72" y2="60.96" width="0.1524" layer="91"/>
-<pinref part="C2" gate="G$1" pin="+"/>
 <wire x1="45.72" y1="60.96" x2="55.88" y2="60.96" width="0.1524" layer="91"/>
 <wire x1="55.88" y1="60.96" x2="58.42" y2="60.96" width="0.1524" layer="91"/>
@@
 <junction x="55.88" y="60.96"/>
 <label x="45.72" y="76.2" size="1.778" layer="95" rot="R90" xref="yes"/>
+<pinref part="C2" gate="G$1" pin="+"/>
 </segment>
 <segment>
@@
 <net name="+3V3" class="0">
 <segment>
-<pinref part="C3" gate="G$1" pin="+"/>
 <wire x1="83.82" y1="40.64" x2="83.82" y2="60.96" width="0.1524" layer="91"/>
 <pinref part="REG_3V3_SPX3940" gate="G$1" pin="OUT"/>
@@
 <junction x="83.82" y="60.96"/>
 <label x="83.82" y="78.74" size="1.778" layer="95" rot="R90" xref="yes"/>
-</segment>
-<segment>
+<pinref part="C3" gate="G$1" pin="+"/>
+</segment>
+<segment>
