File: MicroMouse_Schematics_Final2.brd (EAGLE design)
At the start: 227 x 80 mm, 64 parts

Commit message: Finalized & Ordered PCB with Garber Files
Other:
- board size 227 x 80 mm -> 99.5 x 90.2 mm
Changed lines of the file:
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@@
 <?xml version="1.0" encoding="utf-8"?>
 <!DOCTYPE eagle SYSTEM "eagle.dtd">
-<eagle version="8.6.0">
+<eagle version="8.7.0">
 <drawing>
 <settings>
@@
 <board>
 <plain>
-<wire x1="0" y1="0" x2="227" y2="0" width="0" layer="20"/>
-<wire x1="227" y1="0" x2="227" y2="80" width="0" layer="20"/>
-<wire x1="227" y1="80" x2="0" y2="80" width="0" layer="20"/>
-<wire x1="0" y1="80" x2="0" y2="0" width="0" layer="20"/>
+<wire x1="51.308" y1="-5.08" x2="149.784" y2="-5.08" width="0" layer="20"/>
+<wire x1="149.784" y1="-5.08" x2="149.276" y2="85.08" width="0" layer="20"/>
+<wire x1="149.276" y1="85.08" x2="50.292" y2="85.08" width="0" layer="20"/>
+<wire x1="50.292" y1="85.08" x2="51.308" y2="-5.08" width="0" layer="20"/>
 </plain>
 <attributes>
